File: NaturalKeyboard.kicad_pcb (KiCad board)
At the start: 2 copper layers, 438.1 x 133.3 mm, 233 parts, among them J1 USB_B_Mini, SW1 ESC, SW10 F9, SW100 RALT_125, SW101 FUNC_125, SW102 MENU_125, SW103 RCTRL_125, SW104 Left, SW105 Dn, SW106 Right, SW107 N0_200, SW108 N., SW11 F10, SW12 F11, SW13 F12, SW14 PrtScn, SW15 ScrLk, SW16 Pause, SW17 N=, SW18 N(, SW19 N), SW2 F1, SW20 N<, SW21 `, SW22 1, SW23 2, SW24 3, SW25 4, SW26 5, SW27 6, SW28 7, SW29 8, SW3 F2, SW30 9, SW31 0, SW32 -, SW33 =, SW34 BS_200, SW35 INS, SW36 HOME, SW37 PgUp, SW38 NmLk, SW39 N/, SW4 F3, SW40 N*, SW41 N-, SW42 Tab_150, SW43 Q, SW44 W, SW45 E, SW46 R, SW47 T, SW48 Y, SW49 U, SW5 F4, SW50 I, SW51 O, SW52 P, SW53 [, SW54 ], SW55 \_150, SW56 DEL, SW57 END, SW58 PgDn, SW59 N7, SW6 F5, SW60 N8, SW61 N9, SW62 N+_200V, SW63 Caps_175, SW64 A, SW65 S, SW66 D, SW67 F, SW68 G, SW69 H, SW7 F6, SW70 J, SW71 K, SW72 L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

Commit message: PCB Review Time!
Parts:
- removed R2: 330R, Resistor_SMD:R_1206_3216Metric_Pad1.42x1.75mm_HandSolder
- added C9: 0.1uF, Capacitor_SMD:C_0402_1005Metric, B.Cu at (67.1, 64.1)
- added R6: 22R, Resistor_SMD:R_0402_1005Metric, B.Cu at (72.1, 49.5)
- added R7: 22R, Resistor_SMD:R_0402_1005Metric, B.Cu at (70.6, 49.5)
- C1: footprint Capacitor_SMD:C_0805_2012Metric_Pad1.18x1.45mm_HandSolder -> Capacitor_SMD:C_0402_1005Metric; moved to F.Cu
- C2, C4, C5: footprint Capacitor_SMD:C_0805_2012Metric_Pad1.18x1.45mm_HandSolder -> Capacitor_SMD:C_0402_1005Metric
- C3: footprint Capacitor_SMD:C_0805_2012Metric_Pad1.18x1.45mm_HandSolder -> Capacitor_SMD:C_0402_1005Metric; moved to B.Cu
- C6: value 1uf -> 0.1uF; footprint Capacitor_SMD:C_0805_2012Metric_Pad1.18x1.45mm_HandSolder -> Capacitor_SMD:C_0402_1005Metric
- C7, C8: value 100nf -> 0.1uF; footprint Capacitor_SMD:C_0805_2012Metric_Pad1.18x1.45mm_HandSolder -> Capacitor_SMD:C_0402_1005Metric
- J1: value USB_B_Mini -> USB_C_Receptacle_USB2.0; footprint acheron_Connectors:USB_MiniB_XM7D-0512 -> Connector_USB:USB_C_Receptacle_HRO_TYPE-C-31-M-12
- R1: footprint Resistor_SMD:R_1206_3216Metric_Pad1.42x1.75mm_HandSolder -> Resistor_SMD:R_0402_1005Metric; moved to F.Cu
- R3: value 1k -> 10k; footprint Resistor_SMD:R_1206_3216Metric_Pad1.42x1.75mm_HandSolder -> Resistor_SMD:R_0402_1005Metric; moved to B.Cu
- R4, R5: value 22r -> 5.1k; footprint Resistor_SMD:R_1206_3216Metric_Pad1.42x1.75mm_HandSolder -> Resistor_SMD:R_0402_1005Metric; moved to F.Cu
- SWP1: moved to F.Cu
- U1: moved to B.Cu
- Y1: value 8MHz -> 16Mhz; footprint Crystal:Crystal_SMD_5032-2Pin_5.0x3.2mm_HandSoldering -> Crystal:Crystal_SMD_3225-4Pin_3.2x2.5mm
- moved SWP1 224.6 mm to (71.5, 53.1)
- moved Y1 222.1 mm to (80.1, 61.5), turned to 135 degrees
- moved R3 216.1 mm to (68.6, 66.6), turned to 90 degrees
- moved C1 216.1 mm to (77.2, 52.2), turned to 180 degrees
- moved C2 213.1 mm to (78.5, 63.2), turned to 315 degrees
- moved R1 212.2 mm to (77.2, 50.8)
- moved C3 204.7 mm to (71.5, 55.3), turned to 90 degrees
- moved U1 202.4 mm to (71.9, 61.5), turned to 270 degrees
- moved C4 200.1 mm to (79.0, 58.9), turned to 45 degrees
- moved C5 197.8 mm to (72.6, 55.3), turned to 90 degrees
- moved R4 191.2 mm to (70.1, 40.6), turned to 270 degrees
- moved C7 189.8 mm to (69.1, 56.1), turned to 180 degrees
- moved C6 189.0 mm to (76.6, 57.3), turned to 90 degrees
- moved C8 186.8 mm to (67.1, 58.9), turned to 270 degrees
- moved R5 181.8 mm to (73.2, 40.6), turned to 270 degrees
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Connections:
- net Net-(C3-Pad1) renamed UCAP
- net Net-(R3-Pad2) renamed HWB
- net Net-(U1-Pad42) renamed AREF
- D1 pad 1: Row1 -> Row0A
- D10 pad 1: Row1 -> Row0B
- D100 pad 1: Row6 -> Row5B
- D101 pad 1: Row6 -> Row5A
- D102 pad 1: Row6 -> Row5B
- D103 pad 1: Row6 -> Row5B
- D104 pad 1: Row6 -> Row5A
- D105 pad 1: Row6 -> Row5B
- D106 pad 1: Row6 -> Row5A
- D107 pad 1: Row6 -> Row5B
- D108 pad 1: Row6 -> Row5B
- D11 pad 1: Row1 -> Row0A
- D12 pad 1: Row1 -> Row0B
- D13 pad 1: Row1 -> Row0A
- D14 pad 1: Row1 -> Row0A
- D15 pad 1: Row1 -> Row0B
- D16 pad 1: Row1 -> Row0A
- D17 pad 1: Row1 -> Row0B
- D18 pad 1: Row1 -> Row0A
- D19 pad 1: Row1 -> Row0B
- D2 pad 1: Row1 -> Row0B
- D20 pad 1: Row1 -> Row0A
- D21 pad 1: Row2 -> Row1A
- D22 pad 1: Row2 -> Row1B
- D23 pad 1: Row2 -> Row1A
- D24 pad 1: Row2 -> Row1B
- D25 pad 1: Row2 -> Row1A
- D26 pad 1: Row2 -> Row1B
- D27 pad 1: Row2 -> Row1A
- D28 pad 1: Row2 -> Row1B
- D29 pad 1: Row2 -> Row1A
- D3 pad 1: Row1 -> Row0A
- D30 pad 1: Row2 -> Row1B
- D31 pad 1: Row2 -> Row1A
- D32 pad 1: Row2 -> Row1B
- D33 pad 1: Row2 -> Row1A
- D34 pad 1: Row2 -> Row1B
- D35 pad 1: Row2 -> Row1A
- D36 pad 1: Row2 -> Row1B
- D37 pad 1: Row2 -> Row1A
- D38 pad 1: Row2 -> Row1B
- D39 pad 1: Row2 -> Row1A
- D4 pad 1: Row1 -> Row0B
- D40 pad 1: Row2 -> Row1B
- D41 pad 1: Row2 -> Row1A
- D42 pad 1: Row3 -> Row2A
- D43 pad 1: Row3 -> Row2B
- D44 pad 1: Row3 -> Row2A
- D45 pad 1: Row3 -> Row2B
- D46 pad 1: Row3 -> Row2A
- D47 pad 1: Row3 -> Row2B
- D48 pad 1: Row3 -> Row2A
- D49 pad 1: Row3 -> Row2B
- D5 pad 1: Row1 -> Row0A
- D50 pad 1: Row3 -> Row2A
- D51 pad 1: Row3 -> Row2B
- D52 pad 1: Row3 -> Row2A
- D53 pad 1: Row3 -> Row2B
- D54 pad 1: Row3 -> Row2A
- D55 pad 1: Row3 -> Row2B
- D56 pad 1: Row3 -> Row2A
- D57 pad 1: Row3 -> Row2B
- D58 pad 1: Row3 -> Row2A
- D59 pad 1: Row3 -> Row2B
- D6 pad 1: Row1 -> Row0B
- D60 pad 1: Row3 -> Row2A
- D61 pad 1: Row3 -> Row2B
- D62 pad 1: Row3 -> Row2A
- D63 pad 1: Row4 -> Row3A
- D64 pad 1: Row4 -> Row3B
- D65 pad 1: Row4 -> Row3A
- D66 pad 1: Row4 -> Row3B
- D67 pad 1: Row4 -> Row3A
- D68 pad 1: Row4 -> Row3B
- D69 pad 1: Row4 -> Row3A
- D7 pad 1: Row1 -> Row0A
- D70 pad 1: Row4 -> Row3B
- D71 pad 1: Row4 -> Row3A
- D72 pad 1: Row4 -> Row3B
- D73 pad 1: Row4 -> Row3A
- D74 pad 1: Row4 -> Row3B
- D75 pad 1: Row4 -> Row3A
- D76 pad 1: Row4 -> Row3B
- D77 pad 1: Row4 -> Row3A
- D78 pad 1: Row4 -> Row3B
- D79 pad 1: Row5 -> Row4A
- D8 pad 1: Row1 -> Row0B
- D80 pad 1: Row5 -> Row4B
- D81 pad 1: Row5 -> Row4A
- D82 pad 1: Row5 -> Row4B
- D83 pad 1: Row5 -> Row4A
- D84 pad 1: Row5 -> Row4B
- D85 pad 1: Row5 -> Row4A
- D86 pad 1: Row5 -> Row4B
- D87 pad 1: Row5 -> Row4A
- D88 pad 1: Row5 -> Row4B
- D89 pad 1: Row5 -> Row4A
- D9 pad 1: Row1 -> Row0A
- D90 pad 1: Row5 -> Row4B
- D91 pad 1: Row5 -> Row4B
- D92 pad 1: Row5 -> Row4B
- D93 pad 1: Row5 -> Row4A
- D94 pad 1: Row5 -> Row4B
- D95 pad 1: Row5 -> Row4A
- D96 pad 1: Row6 -> Row5A
- D97 pad 1: Row6 -> Row5B
- D98 pad 1: Row6 -> Row5A
- D99 pad 1: Row6 -> Row5B
- R4 pad 1: Net-(J1-Pad3) -> GND
- R4 pad 2: USB_D+ -> CC1
- R5 pad 1: Net-(J1-Pad2) -> GND
- R5 pad 2: USB_D- -> CC2
- SW1 pad 1: Col1 -> Col0
- SW10 pad 1: Col10 -> Col4
- SW100 pad 1: Col8 -> Col3
- SW101 pad 1: Col9 -> Col4
- SW102 pad 1: Col10 -> Col4
- SW103 pad 1: Col12 -> Col5
- SW104 pad 1: Col15 -> Col7
- SW105 pad 1: Col16 -> Col7
- SW106 pad 1: Col17 -> Col8
- SW107 pad 1: Col18 -> Col8
- SW108 pad 1: Col20 -> Col9
- SW11 pad 1: Col11 -> Col5
- SW12 pad 1: Col12 -> Col5
- SW13 pad 1: Col13 -> Col6
- SW14 pad 1: Col15 -> Col7
- SW15 pad 1: Col16 -> Col7
- SW16 pad 1: Col17 -> Col8
- SW17 pad 1: Col18 -> Col8
- SW18 pad 1: Col19 -> Col9
- SW19 pad 1: Col20 -> Col9
- SW2 pad 1: Col2 -> Col0
- SW20 pad 1: Col21 -> Col10
- SW21 pad 1: Col1 -> Col0
- SW22 pad 1: Col2 -> Col0
- SW23 pad 1: Col3 -> Col1
- SW24 pad 1: Col4 -> Col1
- SW25 pad 1: Col5 -> Col2
- SW26 pad 1: Col6 -> Col2
- SW27 pad 1: Col7 -> Col3
- SW28 pad 1: Col8 -> Col3
- SW29 pad 1: Col9 -> Col4
- SW3 pad 1: Col3 -> Col1
- SW30 pad 1: Col10 -> Col4
- SW31 pad 1: Col11 -> Col5
- SW32 pad 1: Col12 -> Col5
- SW33 pad 1: Col13 -> Col6
- SW34 pad 1: Col14 -> Col6
- SW35 pad 1: Col15 -> Col7
- SW36 pad 1: Col16 -> Col7
- SW37 pad 1: Col17 -> Col8
- SW38 pad 1: Col18 -> Col8
- SW39 pad 1: Col19 -> Col9
- SW4 pad 1: Col4 -> Col1
- SW40 pad 1: Col20 -> Col9
- SW41 pad 1: Col21 -> Col10
- SW42 pad 1: Col1 -> Col0
- SW43 pad 1: Col2 -> Col0
- SW44 pad 1: Col3 -> Col1
- SW45 pad 1: Col4 -> Col1
- SW46 pad 1: Col5 -> Col2
- SW47 pad 1: Col6 -> Col2
- SW48 pad 1: Col7 -> Col3
- SW49 pad 1: Col8 -> Col3
- SW5 pad 1: Col5 -> Col2
- SW50 pad 1: Col9 -> Col4
- SW51 pad 1: Col10 -> Col4
- SW52 pad 1: Col11 -> Col5
- SW53 pad 1: Col12 -> Col5
- SW54 pad 1: Col13 -> Col6
- SW55 pad 1: Col14 -> Col6
- SW56 pad 1: Col15 -> Col7
- SW57 pad 1: Col16 -> Col7
- SW58 pad 1: Col17 -> Col8
- SW59 pad 1: Col18 -> Col8
- SW6 pad 1: Col6 -> Col2
- SW60 pad 1: Col19 -> Col9
- SW61 pad 1: Col20 -> Col9
- SW62 pad 1: Col21 -> Col10
- SW63 pad 1: Col1 -> Col0
- SW64 pad 1: Col2 -> Col0
- SW65 pad 1: Col3 -> Col1
- SW66 pad 1: Col4 -> Col1
- SW67 pad 1: Col5 -> Col2
- SW68 pad 1: Col6 -> Col2
- SW69 pad 1: Col7 -> Col3
- SW7 pad 1: Col7 -> Col3
- SW70 pad 1: Col8 -> Col3
- SW71 pad 1: Col9 -> Col4
- SW72 pad 1: Col10 -> Col4
- SW73 pad 1: Col11 -> Col5
- SW74 pad 1: Col12 -> Col5
- SW75 pad 1: Col13 -> Col6
- SW76 pad 1: Col18 -> Col8
- SW77 pad 1: Col19 -> Col9
- SW78 pad 1: Col20 -> Col9
- SW79 pad 1: Col1 -> Col0
- SW8 pad 1: Col8 -> Col3
- SW80 pad 1: Col2 -> Col0
- SW81 pad 1: Col3 -> Col1
- SW82 pad 1: Col4 -> Col1
- SW83 pad 1: Col5 -> Col2
- SW84 pad 1: Col6 -> Col2
- SW85 pad 1: Col7 -> Col3
- SW86 pad 1: Col8 -> Col3
- SW87 pad 1: Col9 -> Col4
- SW88 pad 1: Col10 -> Col4
- SW89 pad 1: Col11 -> Col5
- SW9 pad 1: Col9 -> Col4
- SW90 pad 1: Col12 -> Col5
- SW91 pad 1: Col16 -> Col7
- SW92 pad 1: Col18 -> Col8
- SW93 pad 1: Col19 -> Col9
- SW94 pad 1: Col20 -> Col9
- SW95 pad 1: Col21 -> Col10
- SW96 pad 1: Col1 -> Col0
- SW97 pad 1: Col2 -> Col0
- SW98 pad 1: Col3 -> Col1
- SW99 pad 1: Col6 -> Col2
- SWP1 pad 1: Net-(R2-Pad1) -> RST
- SWP1 pad 2: RST -> GND
- U1 pad 10: Net-(U1-Pad10) -> Col9
- U1 pad 11: Net-(U1-Pad11) -> Col8
- U1 pad 12: Net-(U1-Pad12) -> Col7
- U1 pad 18: Net-(U1-Pad18) -> Col6
- U1 pad 19: Net-(U1-Pad19) -> Col5
- U1 pad 20: Net-(U1-Pad20) -> Col4
- U1 pad 21: Net-(U1-Pad21) -> Col3
- U1 pad 22: Net-(U1-Pad22) -> Col2
- U1 pad 25: Net-(U1-Pad25) -> Col1
- U1 pad 26: Net-(U1-Pad26) -> Row1B
- U1 pad 28: Net-(U1-Pad28) -> Col0
- U1 pad 29: Net-(U1-Pad29) -> Row1A
- U1 pad 3: USB_D- -> MCU_D-
- U1 pad 30: Net-(U1-Pad30) -> Row2B
- U1 pad 31: Net-(U1-Pad31) -> Row2A
- U1 pad 32: Net-(U1-Pad32) -> Row3B
- U1 pad 36: Net-(U1-Pad36) -> Row3A
- U1 pad 37: Net-(U1-Pad37) -> Row4B
- U1 pad 38: Net-(U1-Pad38) -> Row4A
- U1 pad 39: Net-(U1-Pad39) -> Row5B
- U1 pad 4: USB_D+ -> MCU_D+
- U1 pad 40: Net-(U1-Pad40) -> Row5A
- U1 pad 41: Net-(U1-Pad41) -> Row0A
- U1 pad 8: Net-(U1-Pad8) -> Row0B
- U1 pad 9: Net-(U1-Pad9) -> Col10
- Y1 pad 2: XTAL2 -> GND
Routing:
- net Row5B: track 0.00 -> 515.4 mm
- net Row4A: track 0.00 -> 514.9 mm
- net Row4B: track 0.00 -> 492.7 mm
- net Row2A: track 0.00 -> 473.5 mm
- net Row3B: track 0.00 -> 470.8 mm
- net Row3A: track 0.00 -> 465.3 mm
- net Row5A: track 0.00 -> 462.1 mm
- net Row1A: track 0.00 -> 461.7 mm
- net Row2B: track 0.00 -> 450.0 mm
- net Col9: track 159.4 -> 582.3 mm
- net Row0A: track 0.00 -> 418.2 mm, vias 0 -> 2
- net Col8: track 151.8 -> 565.4 mm
- net Row2: track 410.9 -> 0.00 mm
- net Row1: track 409.6 -> 0.00 mm
- net Row5: track 408.5 -> 0.00 mm
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- added copper zone on B.Cu, net GND
- added copper zone on F.Cu, net GND
- added copper zone on B.Cu, net SHIELD
