File: NaturalKeyboard.sch (KiCad schematic (older format))
At the start: 236 parts, among them J1 USB_C_Receptacle_USB2.0, SW1 ESC, SW10 F9, SW100 RALT_125, SW101 FUNC_125, SW102 MENU_125, SW103 RCTRL_125, SW104 Left, SW105 Dn, SW106 Right, SW107 N0_200, SW108 N., SW11 F10, SW12 F11, SW13 F12, SW14 PrtScn, SW15 ScrLk, SW16 Pause, SW17 N=, SW18 N(, SW19 N), SW2 F1, SW20 N<, SW21 `, SW22 1, SW23 2, SW24 3, SW25 4, SW26 5, SW27 6, SW28 7, SW29 8, SW3 F2, SW30 9, SW31 0, SW32 -, SW33 =, SW34 BS_200, SW35 INS, SW36 HOME, SW37 PgUp, SW38 NmLk, SW39 N/, SW4 F3, SW40 N*, SW41 N-, SW42 Tab_150, SW43 Q, SW44 W, SW45 E, SW46 R, SW47 T, SW48 Y, SW49 U, SW5 F4, SW50 I, SW51 O, SW52 P, SW53 [, SW54 ], SW55 \\_150, SW56 DEL, SW57 END, SW58 PgDn, SW59 N7, SW6 F5, SW60 N8, SW61 N9, SW62 N+_200V, SW63 Caps_175, SW64 A, SW65 S, SW66 D, SW67 F, SW68 G, SW69 H, SW7 F6, SW70 J, SW71 K, SW72 L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

Commit message: PCB Review Time!
Parts:
- removed R2: 330R, Resistor_SMD:R_1206_3216Metric_Pad1.42x1.75mm_HandSolder, symbol Device:R_Small
- C1, C2, C3, C4, C5, C6, C7, C8, C9: footprint Capacitor_SMD:C_0805_2012Metric_Pad1.18x1.45mm_HandSolder -> Capacitor_SMD:C_0402_1005Metric
- R1, R4, R5, R6, R7: footprint Resistor_SMD:R_1206_3216Metric_Pad1.42x1.75mm_HandSolder -> Resistor_SMD:R_0402_1005Metric
- R3: value 1k -> 10k; footprint Resistor_SMD:R_1206_3216Metric_Pad1.42x1.75mm_HandSolder -> Resistor_SMD:R_0402_1005Metric
Connections:
- net Col11 is gone; now on net Col5: SW11.1 (Col), SW31.1 (Col), SW52.1 (Col), SW73.1 (Col), SW89.1 (Col)
- net Col12 is gone; now on net Col5: SW103.1 (Col), SW12.1 (Col), SW32.1 (Col), SW53.1 (Col), SW74.1 (Col), SW90.1 (Col)
- net Col13 is gone; now on net Col6: SW13.1 (Col), SW33.1 (Col), SW54.1 (Col), SW75.1 (Col)
- net Col14 is gone; now on net Col6: SW34.1 (Col), SW55.1 (Col)
- net Col15 is gone; now on net Col7: SW104.1 (Col), SW14.1 (Col), SW35.1 (Col), SW56.1 (Col)
- net Col16 is gone; now on net Col7: SW105.1 (Col), SW15.1 (Col), SW36.1 (Col), SW57.1 (Col), SW91.1 (Col)
- net Col17 is gone; now on net Col8: SW106.1 (Col), SW16.1 (Col), SW37.1 (Col), SW58.1 (Col)
- net Col18 is gone; now on net Col8: SW107.1 (Col), SW17.1 (Col), SW38.1 (Col), SW59.1 (Col), SW76.1 (Col), SW92.1 (Col)
- net Col19 is gone; now on net Col9: SW18.1 (Col), SW39.1 (Col), SW60.1 (Col), SW77.1 (Col), SW93.1 (Col)
- net Col20 is gone; now on net Col9: SW108.1 (Col), SW19.1 (Col), SW40.1 (Col), SW61.1 (Col), SW78.1 (Col), SW94.1 (Col)
- net Col21 is gone; now on net Col10: SW20.1 (Col), SW41.1 (Col), SW62.1 (Col), SW95.1 (Col)
- net Col1: now also SW23.1 (Col), SW24.1 (Col), SW3.1 (Col), SW4.1 (Col), SW44.1 (Col), SW45.1 (Col), SW65.1 (Col), SW66.1 (Col), SW81.1 (Col), SW82.1 (Col), SW98.1 (Col), U1.25 (PD4); no longer SW1.1 (Col), SW21.1 (Col), SW42.1 (Col), SW63.1 (Col), SW79.1 (Col), SW96.1 (Col)
- net Col10: now also U1.9 (PB1); no longer SW10.1 (Col), SW102.1 (Col), SW30.1 (Col), SW51.1 (Col), SW72.1 (Col), SW88.1 (Col)
- net Col2: now also SW25.1 (Col), SW26.1 (Col), SW46.1 (Col), SW47.1 (Col), SW5.1 (Col), SW6.1 (Col), SW67.1 (Col), SW68.1 (Col), SW83.1 (Col), SW84.1 (Col), SW99.1 (Col), U1.22 (PD5); no longer SW2.1 (Col), SW22.1 (Col), SW43.1 (Col), SW64.1 (Col), SW80.1 (Col), SW97.1 (Col)
- net Col3: now also SW100.1 (Col), SW27.1 (Col), SW28.1 (Col), SW48.1 (Col), SW49.1 (Col), SW69.1 (Col), SW7.1 (Col), SW70.1 (Col), SW8.1 (Col), SW85.1 (Col), SW86.1 (Col), U1.21 (PD3); no longer SW23.1 (Col), SW3.1 (Col), SW44.1 (Col), SW65.1 (Col), SW81.1 (Col), SW98.1 (Col)
- net Col4: now also SW10.1 (Col), SW101.1 (Col), SW102.1 (Col), SW29.1 (Col), SW30.1 (Col), SW50.1 (Col), SW51.1 (Col), SW71.1 (Col), SW72.1 (Col), SW87.1 (Col), SW88.1 (Col), SW9.1 (Col), U1.20 (PD2); no longer SW24.1 (Col), SW4.1 (Col), SW45.1 (Col), SW66.1 (Col), SW82.1 (Col)
- net Col5: now also U1.19 (PD1); no longer SW25.1 (Col), SW46.1 (Col), SW5.1 (Col), SW67.1 (Col), SW83.1 (Col)
- net Col6: now also U1.18 (PD0); no longer SW26.1 (Col), SW47.1 (Col), SW6.1 (Col), SW68.1 (Col), SW84.1 (Col), SW99.1 (Col)
- net Col7: now also U1.12 (PB7); no longer SW27.1 (Col), SW48.1 (Col), SW69.1 (Col), SW7.1 (Col), SW85.1 (Col)
- net Col8: now also U1.11 (PB3); no longer SW100.1 (Col), SW28.1 (Col), SW49.1 (Col), SW70.1 (Col), SW8.1 (Col), SW86.1 (Col)
- net Col9: now also U1.10 (PB2); no longer SW101.1 (Col), SW29.1 (Col), SW50.1 (Col), SW71.1 (Col), SW87.1 (Col), SW9.1 (Col)
- net GND: now also SWP1.2
- net RST: now also SWP1.1; no longer SWP1.2
- net XTAL2: now reaches C4.1, U1.16 (XTAL2), Y1.3
- net XTAL1: now reaches C2.1, U1.17 (XTAL1), Y1.1
- net Row1B: now reaches U1.26 (PD6)
- net Row1B: now also D22.1 (K), D24.1 (K), D26.1 (K), D28.1 (K), D30.1 (K), D32.1 (K), D34.1 (K), D36.1 (K), D38.1 (K), D40.1 (K)
- net Col0: now reaches U1.28 (PB4)
- net Col0: now also SW1.1 (Col), SW2.1 (Col), SW21.1 (Col), SW22.1 (Col), SW42.1 (Col), SW43.1 (Col), SW63.1 (Col), SW64.1 (Col), SW79.1 (Col), SW80.1 (Col), SW96.1 (Col), SW97.1 (Col)
- net Row1A: now reaches U1.29 (PB5)
- net Row1A: now also D21.1 (K), D23.1 (K), D25.1 (K), D27.1 (K), D29.1 (K), D31.1 (K), D33.1 (K), D35.1 (K), D37.1 (K), D39.1 (K), D41.1 (K)
- net MCU_D-: now reaches R7.2, U1.3 (D-)
- net Row2B: now reaches U1.30 (PB6)
- net Row2B: now also D43.1 (K), D45.1 (K), D47.1 (K), D49.1 (K), D51.1 (K), D53.1 (K), D55.1 (K), D57.1 (K), D59.1 (K), D61.1 (K)
- net Row2A: now reaches U1.31 (PC6)
- net Row2A: now also D42.1 (K), D44.1 (K), D46.1 (K), D48.1 (K), D50.1 (K), D52.1 (K), D54.1 (K), D56.1 (K), D58.1 (K), D60.1 (K), D62.1 (K)
- net Row3B: now reaches U1.32 (PC7)
- net Row3B: now also D64.1 (K), D66.1 (K), D68.1 (K), D70.1 (K), D72.1 (K), D74.1 (K), D76.1 (K), D78.1 (K)
- net HWB: now reaches R3.2, U1.33 (~HWB~/PE2)
- net Row3A: now reaches U1.36 (PF7)
- net Row3A: now also D63.1 (K), D65.1 (K), D67.1 (K), D69.1 (K), D71.1 (K), D73.1 (K), D75.1 (K), D77.1 (K)
- net Row4B: now reaches U1.37 (PF6)
- net Row4B: now also D80.1 (K), D82.1 (K), D84.1 (K), D86.1 (K), D88.1 (K), D90.1 (K), D91.1 (K), D92.1 (K), D94.1 (K)
- net Row4A: now reaches U1.38 (PF5)
- net Row4A: now also D79.1 (K), D81.1 (K), D83.1 (K), D85.1 (K), D87.1 (K), D89.1 (K), D93.1 (K), D95.1 (K)
- net Row5B: now reaches U1.39 (PF4)
- net Row5B: now also D100.1 (K), D102.1 (K), D103.1 (K), D105.1 (K), D107.1 (K), D108.1 (K), D97.1 (K), D99.1 (K)
- net MCU_D+: now reaches R6.1, U1.4 (D+)
- net Row5A: now reaches U1.40 (PF1)
- net Row5A: now also D101.1 (K), D104.1 (K), D106.1 (K), D96.1 (K), D98.1 (K)
- net Row0A: now reaches U1.41 (PF0)
- net Row0A: now also D1.1 (K), D11.1 (K), D13.1 (K), D14.1 (K), D16.1 (K), D18.1 (K), D20.1 (K), D3.1 (K), D5.1 (K), D7.1 (K), D9.1 (K)
- net AREF: now reaches U1.42 (AREF)
- net UCAP: now reaches C3.1, U1.6 (UCAP)
- net Row0B: now reaches U1.8 (PB0)
- net Row0B: now also D10.1 (K), D12.1 (K), D15.1 (K), D17.1 (K), D19.1 (K), D2.1 (K), D4.1 (K), D6.1 (K), D8.1 (K)
- net CC1: now reaches J1.A5 (CC1), R4.2
- net CC2: now reaches J1.B5 (CC2), R5.2
- net SHIELD: now reaches J1.S1 (SHIELD)
- removed net Row1: D1.1 (K), D10.1 (K), D11.1 (K), D12.1 (K), D13.1 (K), D14.1 (K), D15.1 (K), D16.1 (K), D17.1 (K), D18.1 (K), D19.1 (K), D2.1 (K), D20.1 (K), D3.1 (K), D4.1 (K), D5.1 (K), D6.1 (K), D7.1 (K), D8.1 (K), D9.1 (K)
- removed net Row2: D21.1 (K), D22.1 (K), D23.1 (K), D24.1 (K), D25.1 (K), D26.1 (K), D27.1 (K), D28.1 (K), D29.1 (K), D30.1 (K), D31.1 (K), D32.1 (K), D33.1 (K), D34.1 (K), D35.1 (K), D36.1 (K), D37.1 (K), D38.1 (K), D39.1 (K), D40.1 (K), D41.1 (K)
- removed net Row3: D42.1 (K), D43.1 (K), D44.1 (K), D45.1 (K), D46.1 (K), D47.1 (K), D48.1 (K), D49.1 (K), D50.1 (K), D51.1 (K), D52.1 (K), D53.1 (K), D54.1 (K), D55.1 (K), D56.1 (K), D57.1 (K), D58.1 (K), D59.1 (K), D60.1 (K), D61.1 (K), D62.1 (K)
- removed net Row4: D63.1 (K), D64.1 (K), D65.1 (K), D66.1 (K), D67.1 (K), D68.1 (K), D69.1 (K), D70.1 (K), D71.1 (K), D72.1 (K), D73.1 (K), D74.1 (K), D75.1 (K), D76.1 (K), D77.1 (K), D78.1 (K)
- removed net Row5: D79.1 (K), D80.1 (K), D81.1 (K), D82.1 (K), D83.1 (K), D84.1 (K), D85.1 (K), D86.1 (K), D87.1 (K), D88.1 (K), D89.1 (K), D90.1 (K), D91.1 (K), D92.1 (K), D93.1 (K), D94.1 (K), D95.1 (K)
- removed net Row6: D100.1 (K), D101.1 (K), D102.1 (K), D103.1 (K), D104.1 (K), D105.1 (K), D106.1 (K), D107.1 (K), D108.1 (K), D96.1 (K), D97.1 (K), D98.1 (K), D99.1 (K)
- no-connect marks 4 -> 3
Other:
- note added: "*UGND must route to USB Ground"
- note added: "DFU Pulldown"
- moved on the sheet: C1, C2, C3, C4, C5, C6, C7, C8, C9, D100, D101, D102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
